Commit message: feat(sim_webots_driver): enhance PR2 robot simulation setup
- Updated .gitignore to include scene_info.json and frames_*.
- Added build.sh and run.sh scripts for building and launching the simulation.
- Expanded README.md with installation instructions and features of the PR2 robot.
- Enhanced package.xml with additional dependencies for navigation and visualization.
- Introduced nav2_params.yaml for navigation configuration and ranger_nav2.rviz for RViz visualization.
- Implemented core functionality in sim_webots_driver.py to support PR2's 8-wheel drive and laser scanning.
- Added URDF model for the PR2 robot and integrated it into the simulation environment.

File: driver/sim_webots_driver/src/swd/resource/ranger.urdf (robot description, URDF)
Before this commit: robot ranger, 0 links, 0 joints
Links:
- added link base_footprint
- added link base_laser_link; visual cylinder length=0.1 radius=0.05
- added link base_link; collision box size=0.6 0.4 0.2; visual box size=0.6 0.4 0.2
- added link laser_tilt_link; visual cylinder length=0.08 radius=0.03
Joints:
- added joint base_footprint_joint: type fixed, parent base_footprint, child base_link, origin xyz=0 0 0.1 rpy=0 0 0
- added joint base_laser_joint: type fixed, parent base_link, child base_laser_link, origin xyz=0.3 0 0.15 rpy=0 0 0
- added joint laser_tilt_joint: type fixed, parent base_link, child laser_tilt_link, origin xyz=0.2 0 0.2 rpy=0 0.3 0

Commit message: feat(sim_webots_driver): rename robot to ranger and update URDF configuration

File: driver/sim_webots_driver/src/swd/resource/ranger.urdf (robot description, URDF)
Before this commit: robot ranger, 4 links, 3 joints
Links:
- removed link base_footprint
- removed link base_laser_link
- removed link base_link
- removed link laser_tilt_link
Joints:
- removed joint base_footprint_joint
- removed joint base_laser_joint
- removed joint laser_tilt_joint
