Commit message: fix(webots): co-locate the depth camera with the colour camera
The stock Astra places the range finder 26 mm beside the colour camera,
yet the driver advertises the stream as depth_registered and RTAB-Map
reprojects it with the colour camera_info. At 1 m that parallax is about
12 px, so every visual loop closure was rejected with zero inliers and
only scan proximity ever corrected drift. Both devices already share a
field of view and resolution, so co-locate them in a deployment-owned
PROTO and zero the matching URDF offset.

Assisted-by: Claude Code:claude-fable-5

File: examples/webots/sim/ros_ws/src/eaios_webots/resource/tiago_full_webots.urdf (robot description, URDF)
Before this commit: robot TIAGo Full Webots, 54 links, 53 joints
Joints:
- joint head_front_camera_depth_joint: origin xyz=0.0 0.025 0.0 rpy=0 0 0 -> xyz=0.0 0.0 0.0 rpy=0 0 0

File: examples/webots/sim/ros_ws/src/eaios_webots/resource/tiago_webots.urdf (robot description, URDF)
Before this commit: robot Tiago Webots, 39 links, 38 joints
Joints:
- joint head_front_camera_depth_joint: origin xyz=0.0 0.025 0.0 rpy=0 0 0 -> xyz=0.0 0.0 0.0 rpy=0 0 0
